Commit message: URDF 建模 和 关节节点发布

File: ROS2_Test/Code/10_URDF_model/install/urdf_robot_create/share/urdf_robot_create/urdf/robot_base.urdf (robot description, URDF)
Before this commit: robot fishbot, 3 links, 2 joints
Links:
- added link base_footprint
- added link caster_link; visual sphere radius=0.016
- added link left_wheel_link; visual cylinder length=0.04 radius=0.032
- added link right_wheel_link; visual cylinder length=0.04 radius=0.032
Joints:
- added joint base_joint: type fixed, parent base_footprint, child base_link, origin xyz=0.0 0.0 0.076 rpy=0 0 0
- added joint caster_joint: type fixed, parent base_link, child caster_link, origin xyz=0.06 0.0 -0.076
- added joint left_wheel_joint: type continuous, parent base_link, child left_wheel_link, origin xyz=-0.02 0.10 -0.06, axis 0 1 0
- added joint right_wheel_joint: type continuous, parent base_link, child right_wheel_link, origin xyz=-0.02 -0.10 -0.06, axis 0 1 0
